Commit message: Update PROVA.urdf.xacro
URDF_NO_WARNING

File: Git_Manuel/URDF/PROVA.urdf.xacro (robot description, xacro)
@@ -1 +1,396 @@
-dwcewefe
+<?xml version="1.0" ?>
+<!-- =================================================================================== -->
+<!-- |    This document was autogenerated by xacro from /home/robotics/ws_moveit/src/urdf/test_arm_gazebo.urdf.xacro | -->
+<!-- |    EDITING THIS FILE BY HAND IS NOT RECOMMENDED                                 | -->
+<!-- =================================================================================== -->
+<robot name="ros_project">
+    <link name="world" />
+    <joint name="base_joint" type="fixed">
+        <parent link="world" />
+        <child link="base_link" />
+        <origin xyz="0 0 0" />
+    </joint>
+    <link name="base_link">
+        <visual>
+            <geometry>
+                <cylinder length="0.1" radius="0.2" />
+            </geometry>
+            <origin xyz="0 0 0.05" />
+        </visual>
+        <collision>
+            <geometry>
+                <cylinder length="0.1" radius="0.2" />
+            </geometry>
+            <origin xyz="0 0 0.05" />
+        </collision>
+        <inertial>
+            <mass value="1" />
+            <inertia ixx="1.0" ixy="0.0" ixz="0.0" iyy="1.0" iyz="0.0" izz="1.0" />
+            <origin xyz="0 0 0" rpy="0 0 0" />
+        </inertial>
+    </link>
+    <link name="joint1">
+        <visual>
+            <geometry>
+                <cylinder length="0.1" radius="0.05" />
+            </geometry>
+            <origin rpy="0 0 0" xyz="0 0 0" />
+        </visual>
+        <collision>
+            <geometry>
+                <cylinder length="0.1" radius="0.05" />
+            </geometry>
+            <origin rpy="0 0 0" xyz="0 0 0" />
+        </collision>
+        <inertial>
+            <mass value="1" />
+            <inertia ixx="1.0" ixy="0.0" ixz="0.0" iyy="1.0" iyz="0.0" izz="1.0" />
+            <origin xyz="0 0 0" rpy="0 0 0" />
+        </inertial>
+    </link>
+    <joint name="l0_to_j1" type="continuous">
+        <axis rpy="0 0 0" xyz="0 0 1" />
+        <parent link="base_link" />
+        <child link="joint1" />
+        <origin rpy="0 0 0" xyz="0 0 0.15000000000000002" />
+    </joint>
+    <transmission name="shoulder_yaw">
+        <type>transmission_interface/SimpleTransmission</type>
+        <joint name="l0_to_j1">
+            <hardwareInterface>hardware_interface/PositionJointInterface</hardwareInterface>
+        </joint>
+        <actuator name="$shoulder_yaw_motor">
+            <mechanicalReduction>1</mechanicalReduction>
+            <hardwareInterface>hardware_interface/EffortJointInterface</hardwareInterface>
+        </actuator>
+    </transmission>
+    <link name="link1">
+        <visual>
+            <geometry>
+                <box size="0.1 0.1 0.2" />
+            </geometry>
+            <origin rpy="1.57 0 0" xyz="0 -0.15000000000000002 0" />
+        </visual>
+        <collision>
+            <geometry>
+                <box size="0.1 0.1 0.2" />
+            </geometry>
+            <origin rpy="1.57 0 0" xyz="0 -0.15000000000000002 0" />
+        </collision>
+        <inertial>
+            <mass value="1" />
+            <inertia ixx="1.0" ixy="0.0" ixz="0.0" iyy="1.0" iyz="0.0" izz="1.0" />
+            <origin xyz="0 0 0" rpy="0 0 0" />
+        </inertial>
+    </link>
+    <joint name="j1_to_l1" type="fixed">
+        <parent link="joint1" />
+        <child link="link1" />
+        <origin rpy="1.57 0 0" xyz="0 0 0.29" />
+    </joint>
+    <link name="joint2">
+        <visual>
+            <geometry>
+                <cylinder length="0.1" radius="0.05" />
+            </geometry>
+            <origin rpy="0 0 0" xyz="0 0 0" />
+        </visual>
+        <collision>
+            <geometry>
+                <cylinder length="0.1" radius="0.05" />
+            </geometry>
+            <origin rpy="0 0 0" xyz="0 0 0" />
+        </collision>
+        <inertial>
+            <mass value="1" />
+            <inertia ixx="1.0" ixy="0.0" ixz="0.0" iyy="1.0" iyz="0.0" izz="1.0" />
+            <origin xyz="0 0 0" rpy="0 0 0" />
+        </inertial>
+    </link>
+    <joint name="l1_to_j2" type="revolute">
+        <axis rpy="0 0 0" xyz="0 0 1" />
+        <limit effort="1000" lower="0" upper="3.14" velocity="0.5" />
+        <parent link="link1" />
+        <child link="joint2" />
+        <origin rpy="0 0 0" xyz="0 0 0" />
+    </joint>
+    <transmission name="shoulder_roll">
+        <type>transmission_interface/SimpleTransmission</type>
+        <joint name="l1_to_j2">
+            <hardwareInterface>hardware_interface/PositionJointInterface</hardwareInterface>
+        </joint>
+        <actuator name="$shoulder_roll_motor">
+            <mechanicalReduction>1</mechanicalReduction>
+            <hardwareInterface>hardware_interface/EffortJointInterface</hardwareInterface>
+        </actuator>
+    </transmission>
+    <link name="link2">
+        <visual>
+            <geometry>
+                <box size="0.1 0.1 0.2" />
+            </geometry>
+            <origin rpy="0 1.57 0" xyz="-0.15000000000000002 0 0" />
+        </visual>
+        <collision>
+            <geometry>
+                <box size="0.1 0.1 0.2" />
+            </geometry>
+            <origin rpy="0 1.57 0" xyz="-0.15000000000000002 0 0" />
+        </collision>
+        <inertial>
+            <mass value="1" />
+            <inertia ixx="1.0" ixy="0.0" ixz="0.0" iyy="1.0" iyz="0.0" izz="1.0" />
+            <origin xyz="0 0 0" rpy="0 0 0" />
+        </inertial>
+    </link>
+    <joint name="j2_to_l2" type="fixed">
+        <parent link="joint2" />
+        <child link="link2" />
+        <origin rpy="0 0 0" xyz="0.30000000000000004 0 0" />
+    </joint>
+    <link name="joint3">
+        <visual>
+            <geometry>
+                <cylinder length="0.1" radius="0.05" />
+            </geometry>
+            <origin rpy="0 0 0" xyz="0 0 0" />
+        </visual>
+        <collision>
+            <geometry>
+                <cylinder length="0.1" radius="0.05" />
+            </geometry>
+            <origin rpy="0 0 0" xyz="0 0 0" />
+        </collision>
+        <inertial>
+            <mass value="1" />
+            <inertia ixx="1.0" ixy="0.0" ixz="0.0" iyy="1.0" iyz="0.0" izz="1.0" />
+            <origin xyz="0 0 0" rpy="0 0 0" />
+        </inertial>
+    </link>
+    <joint name="l2_to_j3" type="revolute">
+        <axis rpy="0 0 0" xyz="0 0 1" />
+        <limit effort="1000" lower="0" upper="3.14" velocity="0.5" />
+        <parent link="link2" />
+        <child link="joint3" />
+        <origin rpy="0 0 0" xyz="0 0 0" />
+    </joint>
+    <transmission name="elbow">
+        <type>transmission_interface/SimpleTransmission</type>
+        <joint name="l2_to_j3">
+            <hardwareInterface>hardware_interface/PositionJointInterface</hardwareInterface>
+        </joint>
+        <actuator name="$elbow_motor">
+            <mechanicalReduction>1</mechanicalReduction>
+            <hardwareInterface>hardware_interface/EffortJointInterface</hardwareInterface>
+        </actuator>
+    </transmission>
+    <link name="link3">
+        <visual>
+            <geometry>
+                <box size="0.1 0.1 0.2" />
+            </geometry>
+            <origin rpy="0 0 0" xyz="0 0 0.15000000000000002" />
+        </visual>
+        <collision>
+            <geometry>
+                <box size="0.1 0.1 0.2" />
+            </geometry>
+            <origin rpy="0 0 0" xyz="0 0.15000000000000002 0" />
+        </collision>
+        <inertial>
+            <mass value="1" />
+            <inertia ixx="1.0" ixy="0.0" ixz="0.0" iyy="1.0" iyz="0.0" izz="1.0" />
+            <origin xyz="0 0 0" rpy="0 0 0" />
+        </inertial>
+    </link>
+    <joint name="j3_to_l3" type="fixed">
+        <parent link="joint3" />
+        <child link="link3" />
+        <origin rpy="1.57 0 0" xyz="0 0 0" />
+    </joint>
+    <link name="joint4">
+        <visual>
+            <geometry>
+                <cylinder length="0.1" radius="0.05" />
+            </geometry>
+            <origin rpy="0 0 0" xyz="0 0 0" />
+        </visual>
+        <collision>
+            <geometry>
+                <cylinder length="0.1" radius="0.05" />
+            </geometry>
+            <origin rpy="0 0 0" xyz="0 0 0" />
+        </collision>
+        <inertial>
+            <mass value="1" />
+            <inertia ixx="1.0" ixy="0.0" ixz="0.0" iyy="1.0" iyz="0.0" izz="1.0" />
+            <origin xyz="0 0 0" rpy="0 0 0" />
+        </inertial>
+    </link>
+    <joint name="l3_to_j4" type="revolute">
+        <axis rpy="0 0 0" xyz="0 0 1" />
+        <limit effort="1000" lower="-1.57" upper="1.57" velocity="0.5" />
+        <parent link="link3" />
+        <child link="joint4" />
+        <origin rpy="0 0 0" xyz="0 0 0.30000000000000004" />
+    </joint>
+    <transmission name="wrist_roll">
+        <type>transmission_interface/SimpleTransmission</type>
+        <joint name="l3_to_j4">
+            <hardwareInterface>hardware_interface/PositionJointInterface</hardwareInterface>
+        </joint>
+        <actuator name="$wrist_roll_motor">
+            <mechanicalReduction>1</mechanicalReduction>
+            <hardwareInterface>hardware_interface/EffortJointInterface</hardwareInterface>
+        </actuator>
+    </transmission>
+    <link name="link4">
+        <visual>
+            <geometry>
+                <box size="0.1 0.1 0.2" />
+            </geometry>
+            <origin rpy="1.57 0 0" xyz="0 0.15000000000000002 0" />
+        </visual>
+        <collision>
+            <geometry>
+                <box size="0.1 0.1 0.2" />
+            </geometry>
+            <origin rpy="1.57 0 0" xyz="0 0.15000000000000002 0" />
+        </collision>
+        <inertial>
+            <mass value="1" />
+            <inertia ixx="1.0" ixy="0.0" ixz="0.0" iyy="1.0" iyz="0.0" izz="1.0" />
+            <origin xyz="0 0 0" rpy="0 0 0" />
+        </inertial>
+    </link>
+    <joint name="j4_to_l4" type="fixed">
+        <parent link="joint4" />
+        <child link="link4" />
+        <origin rpy="-1.57 0 0" xyz="0 0 0.30000000000000004" />
+    </joint>
+    <link name="joint5">
+        <visual>
+            <geometry>
+                <cylinder length="0.1" radius="0.05" />
+            </geometry>
+            <origin rpy="0 0 0" xyz="0 0 0" />
+        </visual>
+        <collision>
+            <geometry>
+                <cylinder length="0.1" radius="0.05" />
+            </geometry>
+            <origin rpy="0 0 0" xyz="0 0 0" />
+        </collision>
+        <inertial>
+            <mass value="1" />
+            <inertia ixx="1.0" ixy="0.0" ixz="0.0" iyy="1.0" iyz="0.0" izz="1.0" />
+            <origin xyz="0 0 0" rpy="0 0 0" />
+        </inertial>
+    </link>
+    <joint name="l4_to_j5" type="revolute">
+        <axis rpy="0 0 0" xyz="0 0 1" />
+        <limit effort="1000" lower="-1.57" upper="1.57" velocity="0.5" />
+        <parent link="link4" />
+        <child link="joint5" />
+        <origin rpy="0 0 0" xyz="0 0 0" />
+    </joint>
+    <transmission name="wrist_pitch">
+        <type>transmission_interface/SimpleTransmission</type>
+        <joint name="l4_to_j5">
+            <hardwareInterface>hardware_interface/PositionJointInterface</hardwareInterface>
+        </joint>
+        <actuator name="$wrist_pitch_motor">
+            <mechanicalReduction>1</mechanicalReduction>
+            <hardwareInterface>hardware_interface/EffortJointInterface</hardwareInterface>
+        </actuator>
+    </transmission>
+    <link name="link5">
+        <visual>
+            <geometry>
+                <box size="0.1 0.1 0.2" />
+            </geometry>
+            <origin rpy="0 0 0" xyz="0 0 0.15000000000000002" />
+        </visual>
+        <collision>
+            <geometry>
+                <box size="0.1 0.1 0.2" />
+            </geometry>
+            <origin rpy="0 0 0" xyz="0 0 0.15000000000000002" />
+        </collision>
+        <inertial>
+            <mass value="1" />
+            <inertia ixx="1.0" ixy="0.0" ixz="0.0" iyy="1.0" iyz="0.0" izz="1.0" />
+            <origin xyz="0 0 0" rpy="0 0 0" />
+        </inertial>
+    </link>
+    <joint name="j5_to_l5" type="fixed">
+        <parent link="joint5" />
+        <child link="link5" />
+        <origin rpy="1.57 0 0" xyz="0 0 0" />
+    </joint>
+    <link name="joint6">
+        <visual>
+            <geometry>
+                <cylinder length="0.1" radius="0.05" />
+            </geometry>
+            <origin rpy="0 0 0" xyz="0 0 0" />
+        </visual>
+        <collision>
+            <geometry>
+                <cylinder length="0.1" radius="0.05" />
+            </geometry>
+            <origin rpy="0 0 0" xyz="0 0 0" />
+        </collision>
+        <inertial>
+            <mass value="1" />
+            <inertia ixx="1.0" ixy="0.0" ixz="0.0" iyy="1.0" iyz="0.0" izz="1.0" />
+            <origin xyz="0 0 0" rpy="0 0 0" />
+        </inertial>
+    </link>
+    <joint name="l5_to_j6" type="revolute">
+        <axis rpy="0 0 0" xyz="0 0 1" />
+        <limit effort="1000" lower="-1.57" upper="1.57" velocity="0.5" />
+        <parent link="link5" />
+        <child link="joint6" />
+        <origin rpy="0 0 0" xyz="0 0 0.30000000000000004" />
+    </joint>
+    <transmission name="wrist_yaw">
+        <type>transmission_interface/SimpleTransmission</type>
+        <joint name="l5_to_j6">
+            <hardwareInterface>hardware_interface/PositionJointInterface</hardwareInterface>
+        </joint>
+        <actuator name="$wrist_yaw_motor">
+            <mechanicalReduction>1</mechanicalReduction>
+            <hardwareInterface>hardware_interface/EffortJointInterface</hardwareInterface>
+        </actuator>
+    </transmission>
+    <link name="link6">
+        <visual>
+            <geometry>
+                <box size="0.1 0.1 0.2" />
+            </geometry>
+            <origin rpy="0 0 0" xyz="0 0 -0.1" />
+        </visual>
+        <collision>
+            <geometry>
+                <box size="0.1 0.1 0.2" />
+            </geometry>
+            <origin rpy="0 0 0" xyz="0 0 -0.1" />
+        </collision>
+        <inertial>
+            <mass value="1" />
+            <inertia ixx="1.0" ixy="0.0" ixz="0.0" iyy="1.0" iyz="0.0" izz="1.0" />
+            <origin xyz="0 0 0" rpy="0 0 0" />
+        </inertial>
+    </link>
+    <joint name="j6_to_l6" type="fixed">
+        <parent link="joint6" />
+        <child link="link6" />
+        <origin rpy="0 0 1.57" xyz="0 0 0.25" />
+    </joint>
+    <gazebo>
+        <plugin filename="libgazebo_ros_control.so" name="gazebo_ros_control">
+            <robotNamespace>/</robotNamespace>
+        </plugin>
+    </gazebo>
+</robot>
